Commit message: cleaned up version of xacro

File: robots/a1_description/xacro/robot_rplidar.xacro (robot description, xacro)
@@ -139,8 +139,3 @@
           </inertial>
       </link>
-    <!--<xacro:include filename="$(find velodyne_description)/urdf/VLP-16.urdf.xacro"/>-->
-    <!--<VLP-16 parent="base" name="velodyne" topic="lidar_points" hz="10" samples="1024" gpu="false" lasers="16" max_range="100">-->
-        <!--<origin xyz="0.0075 0.0 0.3025" rpy="0 0 0" />-->
-    <!--</VLP-16>-->
-    <!-- <xacro:stairs stairs="15" xpos="0" ypos="2.0" zpos="0" /> -->
 </robot>
