Commit message: first commit with new Go1 code

File: robots/a1_description/urdf/a1.urdf (robot description, URDF)
Before this commit: robot a1_description, 23 links, 22 joints
Links:
- link trunk: mass 4.713 -> 6.0
Joints:
- joint FL_calf_joint: limit lower=-2.69653369433 upper=-0.916297857297 effort=55 velocity=28.6 -> lower=-2.69653369433 upper=-0.916297857297 effort=33.5 velocity=21
- joint FL_hip_joint: limit lower=-0.802851455917 upper=0.802851455917 effort=20 velocity=52.4 -> lower=-0.802851455917 upper=0.802851455917 effort=33.5 velocity=21; origin xyz=0.183 0.047 0 rpy=0 0 0 -> xyz=0.1805 0.047 0 rpy=0 0 0
- joint FL_thigh_joint: limit lower=-1.0471975512 upper=4.18879020479 effort=55 velocity=28.6 -> lower=-1.0471975512 upper=4.18879020479 effort=33.5 velocity=21; origin xyz=0 0.08505 0 rpy=0 0 0 -> xyz=0 0.0838 0 rpy=0 0 0
- joint FR_calf_joint: limit lower=-2.69653369433 upper=-0.916297857297 effort=55 velocity=28.6 -> lower=-2.69653369433 upper=-0.916297857297 effort=33.5 velocity=21
- joint FR_hip_joint: limit lower=-0.802851455917 upper=0.802851455917 effort=20 velocity=52.4 -> lower=-0.802851455917 upper=0.802851455917 effort=33.5 velocity=21; origin xyz=0.183 -0.047 0 rpy=0 0 0 -> xyz=0.1805 -0.047 0 rpy=0 0 0
- joint FR_thigh_joint: limit lower=-1.0471975512 upper=4.18879020479 effort=55 velocity=28.6 -> lower=-1.0471975512 upper=4.18879020479 effort=33.5 velocity=21; origin xyz=0 -0.08505 0 rpy=0 0 0 -> xyz=0 -0.0838 0 rpy=0 0 0
- joint RL_calf_joint: limit lower=-2.69653369433 upper=-0.916297857297 effort=55 velocity=28.6 -> lower=-2.69653369433 upper=-0.916297857297 effort=33.5 velocity=21
- joint RL_hip_joint: limit lower=-0.802851455917 upper=0.802851455917 effort=20 velocity=52.4 -> lower=-0.802851455917 upper=0.802851455917 effort=33.5 velocity=21; origin xyz=-0.183 0.047 0 rpy=0 0 0 -> xyz=-0.1805 0.047 0 rpy=0 0 0
- joint RL_thigh_joint: limit lower=-1.0471975512 upper=4.18879020479 effort=55 velocity=28.6 -> lower=-1.0471975512 upper=4.18879020479 effort=33.5 velocity=21; origin xyz=0 0.08505 0 rpy=0 0 0 -> xyz=0 0.0838 0 rpy=0 0 0
- joint RR_calf_joint: limit lower=-2.69653369433 upper=-0.916297857297 effort=55 velocity=28.6 -> lower=-2.69653369433 upper=-0.916297857297 effort=33.5 velocity=21
- joint RR_hip_joint: limit lower=-0.802851455917 upper=0.802851455917 effort=20 velocity=52.4 -> lower=-0.802851455917 upper=0.802851455917 effort=33.5 velocity=21; origin xyz=-0.183 -0.047 0 rpy=0 0 0 -> xyz=-0.1805 -0.047 0 rpy=0 0 0
- joint RR_thigh_joint: limit lower=-1.0471975512 upper=4.18879020479 effort=55 velocity=28.6 -> lower=-1.0471975512 upper=4.18879020479 effort=33.5 velocity=21; origin xyz=0 -0.08505 0 rpy=0 0 0 -> xyz=0 -0.0838 0 rpy=0 0 0

File: robots/a1_description/xacro/const.xacro (robot description, xacro)
@@ -1,4 +1,4 @@
 <?xml version="1.0"?>
-<robot name="a1_description" xmlns:xacro="http://www.ros.org/wiki/xacro">
+<robot xmlns:xacro="http://www.ros.org/wiki/xacro">
     <!-- Constants for robot dimensions -->
     <xacro:property name="PI" value="3.1415926535897931"/>
@@ -20,9 +20,9 @@
     <xacro:property name="stick_length" value="0.2"/>
     <!-- kinematic value -->
-    <xacro:property name="thigh_offset" value="0.08505"/>
+    <xacro:property name="thigh_offset" value="0.0838"/>
     <xacro:property name="thigh_length" value="0.2"/>
     <xacro:property name="calf_length" value="0.2"/>
     <!-- leg offset from trunk center value -->
-    <xacro:property name="leg_offset_x" value="0.183"/>
+    <xacro:property name="leg_offset_x" value="0.1805"/>
     <xacro:property name="leg_offset_y" value="0.047"/>
     <xacro:property name="trunk_offset_z" value="0.01675"/>
@@ -33,59 +33,59 @@
     <xacro:property name="hip_max" value="46"/>
     <xacro:property name="hip_min" value="-46"/>
-    <xacro:property name="hip_velocity_max" value="52.4"/>
-    <xacro:property name="hip_torque_max" value="20"/>
+    <xacro:property name="hip_velocity_max" value="21"/>
+    <xacro:property name="hip_torque_max" value="33.5"/>
     <xacro:property name="thigh_max" value="240"/>
     <xacro:property name="thigh_min" value="-60"/>
-    <xacro:property name="thigh_velocity_max" value="28.6"/>
-    <xacro:property name="thigh_torque_max" value="55"/>
+    <xacro:property name="thigh_velocity_max" value="21"/>
+    <xacro:property name="thigh_torque_max" value="33.5"/>
     <xacro:property name="calf_max" value="-52.5"/>
     <xacro:property name="calf_min" value="-154.5"/>
-    <xacro:property name="calf_velocity_max" value="28.6"/>
-    <xacro:property name="calf_torque_max" value="55"/>
-    <!-- dynamics inertial value -->
+    <xacro:property name="calf_velocity_max" value="21"/>
+    <xacro:property name="calf_torque_max" value="33.5"/>
+    <!-- dynamics inertial value        total 13.9kg -->
     <!-- trunk -->
-    <xacro:property name="trunk_mass" value="4.713"/>
-    <xacro:property name="trunk_com_x" value="0.012731"/>
-    <xacro:property name="trunk_com_y" value="0.002186"/>
-    <xacro:property name="trunk_com_z" value="0.000515"/>
-    <xacro:property name="trunk_ixx" value="0.016839930"/>
-    <xacro:property name="trunk_ixy" value="0.000083902"/>
-    <xacro:property name="trunk_ixz" value="0.000597679"/>
-    <xacro:property name="trunk_iyy" value="0.056579028"/>
-    <xacro:property name="trunk_iyz" value="0.000025134"/>
-    <xacro:property name="trunk_izz" value="0.064713601"/>
+    <xacro:property name="trunk_mass" value="6.0"/>
+    <xacro:property name="trunk_com_x" value="0.0000"/>
+    <xacro:property name="trunk_com_y" value="0.0041"/>
+    <xacro:property name="trunk_com_z" value="-0.0005"/>
+    <xacro:property name="trunk_ixx" value="0.0158533"/>
+    <xacro:property name="trunk_ixy" value="-0.0000366"/>
+    <xacro:property name="trunk_ixz" value="-0.0000611"/>
+    <xacro:property name="trunk_iyy" value="0.0377999"/>
+    <xacro:property name="trunk_iyz" value="-0.0000275"/>
+    <xacro:property name="trunk_izz" value="0.0456542"/>
     <!-- hip (left front) -->
-    <xacro:property name="hip_mass" value="0.696"/>
-    <xacro:property name="hip_com_x" value="-0.003311"/>
-    <xacro:property name="hip_com_y" value="0.000635"/>
-    <xacro:property name="hip_com_z" value="0.000031"/>
-    <xacro:property name="hip_ixx" value="0.000469246"/>
-    <xacro:property name="hip_ixy" value="-0.000009409"/>
-    <xacro:property name="hip_ixz" value="-0.000000342"/>
-    <xacro:property name="hip_iyy" value="0.000807490"/>
-    <xacro:property name="hip_iyz" value="-0.000000466"/>
-    <xacro:property name="hip_izz" value="0.000552929"/>
+    <xacro:property name="hip_mass" value="0.595"/>
+    <xacro:property name="hip_com_x" value="-0.003875"/>
+    <xacro:property name="hip_com_y" value="0.001622"/>
+    <xacro:property name="hip_com_z" value="0.000042"/>
+    <xacro:property name="hip_ixx" value="0.000402747"/>
+    <xacro:property name="hip_ixy" value="-0.000008709"/>
+    <xacro:property name="hip_ixz" value="-0.000000297"/>
+    <xacro:property name="hip_iyy" value="0.000691123"/>
+    <xacro:property name="hip_iyz" value="-0.000000545"/>
+    <xacro:property name="hip_izz" value="0.000487919"/>
     <!-- thigh -->
-    <xacro:property name="thigh_mass" value="1.013"/>
-    <xacro:property name="thigh_com_x" value="-0.003237"/>
-    <xacro:property name="thigh_com_y" value="-0.022327"/>
-    <xacro:property name="thigh_com_z" value="-0.027326"/>
-    <xacro:property name="thigh_ixx" value="0.005529065"/>
-    <xacro:property name="thigh_ixy" value="0.000004825"/>
-    <xacro:property name="thigh_ixz" value="0.000343869"/>
-    <xacro:property name="thigh_iyy" value="0.005139339"/>
-    <xacro:property name="thigh_iyz" value="0.000022448"/>
-    <xacro:property name="thigh_izz" value="0.001367788"/>
+    <xacro:property name="thigh_mass" value="0.888"/>
+    <xacro:property name="thigh_com_x" value="-0.003574"/>
+    <xacro:property name="thigh_com_y" value="-0.019529"/>
+    <xacro:property name="thigh_com_z" value="-0.030323"/>
+    <xacro:property name="thigh_ixx" value="0.005251806"/>
+    <xacro:property name="thigh_ixy" value="-0.000002168"/>
+    <xacro:property name="thigh_ixz" value="0.000346889"/>
+    <xacro:property name="thigh_iyy" value="0.005000475"/>
+    <xacro:property name="thigh_iyz" value="-0.000028174"/>
+    <xacro:property name="thigh_izz" value="0.001110200"/>
     <!-- calf -->
-    <xacro:property name="calf_mass" value="0.166"/>
-    <xacro:property name="calf_com_x" value="0.006435"/>
-    <xacro:property name="calf_com_y" value="0.0"/>
-    <xacro:property name="calf_com_z" value="-0.107388"/>
-    <xacro:property name="calf_ixx" value="0.002997972"/>
+    <xacro:property name="calf_mass" value="0.151"/>
+    <xacro:property name="calf_com_x" value="0.007105"/>
+    <xacro:property name="calf_com_y" value="-0.000239"/>
+    <xacro:property name="calf_com_z" value="-0.096933"/>
+    <xacro:property name="calf_ixx" value="0.002344758"/>
     <xacro:property name="calf_ixy" value="0.0"/>
-    <xacro:property name="calf_ixz" value="-0.000141163"/>
-    <xacro:property name="calf_iyy" value="0.003014022"/>
+    <xacro:property name="calf_ixz" value="-0.000141275"/>
+    <xacro:property name="calf_iyy" value="0.002360755"/>
     <xacro:property name="calf_iyz" value="0.0"/>
-    <xacro:property name="calf_izz" value="0.000032426"/>
+    <xacro:property name="calf_izz" value="0.000031158"/>
     <!-- foot -->
     <xacro:property name="foot_mass" value="0.06"/>

File: robots/a1_description/xacro/gazebo.xacro (robot description, xacro)
@@ -1,33 +1,4 @@
 <?xml version="1.0"?>
 <robot>
-    <gazebo>
-    <plugin name="diff_drive_controller" filename="libgazebo_ros_diff_drive.so">
-      <publishWheelTF>true</publishWheelTF>
-      <publishOdomTF>true</publishOdomTF>
-      <alwaysOn>true</alwaysOn>
-      <legacyMode>false</legacyMode>
-      <updateRate>40</updateRate>
-      <leftJoint>left_wheel_joint</leftJoint>
-      <rightJoint>right_wheel_joint</rightJoint>
-      <wheelSeparation>0.5</wheelSeparation>
-      <wheelDiameter>0.3</wheelDiameter>
-      <torque>20</torque>
-      <commandTopic>cmd_vel</commandTopic>
-      <odometryTopic>odom</odometryTopic>
-      <odometryFrame>odom</odometryFrame>
-      <robotBaseFrame>base</robotBaseFrame>
-    </plugin>
-  </gazebo>
-  <gazebo>
-      <plugin name="force_based_move_controller" filename="libgazebo_ros_force_based_move.so">
-        <commandTopic>/cmd_vel_raw</commandTopic>
-        <odometryTopic>odom</odometryTopic>
-        <odometryFrame>odom</odometryFrame>
-        <odometryRate>20.0</odometryRate>
-        <robotBaseFrame>base</robotBaseFrame>
-        <yaw_velocity_p_gain>250</yaw_velocity_p_gain>
-        <publishOdometryTf>1</publishOdometryTf>
-      </plugin>
-    </gazebo>
     <!-- ros_control plugin -->
     <gazebo>

File: robots/a1_description/xacro/robot.xacro (robot description, xacro)
@@ -1,4 +1,5 @@
 <?xml version="1.0"?>
-<robot name="a1_description" xmlns:xacro="http://www.ros.org/wiki/xacro">
+<robot name="a1" xmlns:xacro="http://www.ros.org/wiki/xacro">
+    <xacro:arg name="DEBUG" default="false"/>
     <xacro:include filename="$(find a1_description)/xacro/const.xacro"/>
     <xacro:include filename="$(find a1_description)/xacro/materials.xacro"/>
@@ -121,8 +122,4 @@
         <origin rpy="0 0 0" xyz="${-leg_offset_x} ${leg_offset_y} 0"/>
     </xacro:leg>
-    <xacro:include filename="$(find velodyne_description)/urdf/VLP-16.urdf.xacro"/>
-    <VLP-16 parent="base" name="velodyne" topic="lidar_points" hz="10" samples="1024" gpu="false" lasers="16" max_range="100">
-        <origin xyz="0.0075 0.0 0.3025" rpy="0 0 0" />
-    </VLP-16>
     <!-- <xacro:stairs stairs="15" xpos="0" ypos="2.0" zpos="0" /> -->
 </robot>

File: robots/aliengo_description/xacro/const.xacro (robot description, xacro)
@@ -1,4 +1,4 @@
 <?xml version="1.0"?>
-<robot name="aliengo_description" xmlns:xacro="http://www.ros.org/wiki/xacro">
+<robot xmlns:xacro="http://www.ros.org/wiki/xacro">
     <!-- Constants for robot dimensions -->
     <xacro:property name="PI" value="3.1415926535897931"/>
@@ -20,12 +20,31 @@
     <xacro:property name="stick_length" value="0.2"/>
     <!-- kinematic value -->
-    <xacro:property name="thigh_offset" value="0.083"/>
+    <xacro:property name="thigh_offset" value="0.0868"/>
     <xacro:property name="thigh_length" value="0.25"/>
     <xacro:property name="calf_length" value="0.25"/>
     <!-- leg offset from trunk center value -->
-    <xacro:property name="leg_offset_x" value="0.2399"/>
+    <xacro:property name="leg_offset_x" value="0.2407"/>
     <xacro:property name="leg_offset_y" value="0.051"/>
     <xacro:property name="trunk_offset_z" value="0.01675"/>
     <xacro:property name="hip_offset" value="0.083"/>
+    <!-- offset of link and rotor locations (left front) -->
+    <xacro:property name="hip_offset_x" value="0.2407"/>
+    <xacro:property name="hip_offset_y" value="0.051"/>
+    <xacro:property name="hip_offset_z" value="0.0"/>
+    <xacro:property name="hip_rotor_offset_x" value="0.139985"/>
+    <xacro:property name="hip_rotor_offset_y" value="0.051"/>
+    <xacro:property name="hip_rotor_offset_z" value="0.0"/>
+    <xacro:property name="thigh_offset_x" value="0"/>
+    <xacro:property name="thigh_offset_y" value="0.0868"/>
+    <xacro:property name="thigh_offset_z" value="0.0"/>
+    <xacro:property name="thigh_rotor_offset_x" value="0.0"/>
+    <xacro:property name="thigh_rotor_offset_y" value="0.0298"/>
+    <xacro:property name="thigh_rotor_offset_z" value="0.0"/>
+    <xacro:property name="calf_offset_x" value="0.0"/>
+    <xacro:property name="calf_offset_y" value="0.0"/>
+    <xacro:property name="calf_offset_z" value="-0.25"/>
+    <xacro:property name="calf_rotor_offset_x" value="0.0"/>
+    <xacro:property name="calf_rotor_offset_y" value="-0.0997"/>
+    <xacro:property name="calf_rotor_offset_z" value="0.0"/>
     <!-- joint limits -->
     <xacro:property name="damping" value="0"/>
@@ -34,23 +53,25 @@
     <xacro:property name="hip_position_min" value="${-70*PI/180.0}"/>
     <xacro:property name="hip_velocity_max" value="20"/>
-    <xacro:property name="hip_torque_max" value="44"/>
+    <xacro:property name="hip_torque_max" value="35.278"/>
+    <xacro:property name="thigh_position_max" value="${240*PI/180.0}"/>
+    <xacro:property name="thigh_position_min" value="${-120*PI/180.0}"/>
     <xacro:property name="thigh_velocity_max" value="20"/>
-    <xacro:property name="thigh_torque_max" value="44"/>
+    <xacro:property name="thigh_torque_max" value="35.278"/>
     <xacro:property name="calf_position_max" value="${-37*PI/180.0}"/>
     <xacro:property name="calf_position_min" value="${-159*PI/180.0}"/>
-    <xacro:property name="calf_velocity_max" value="16"/>
-    <xacro:property name="calf_torque_max" value="55"/>
-    <!-- dynamics inertial value -->
+    <xacro:property name="calf_velocity_max" value="15.89"/>
+    <xacro:property name="calf_torque_max" value="44.4"/>
+    <!-- dynamics inertial value        total 23.0kg -->
     <!-- trunk -->
-    <xacro:property name="trunk_mass" value="9.041"/>
-    <xacro:property name="trunk_com_x" value="0.008465"/>
-    <xacro:property name="trunk_com_y" value="0.004045"/>
-    <xacro:property name="trunk_com_z" value="-0.000763"/>
-    <xacro:property name="trunk_ixx" value="0.033260231"/>
-    <xacro:property name="trunk_ixy" value="-0.000451628"/>
-    <xacro:property name="trunk_ixz" value="0.000487603"/>
-    <xacro:property name="trunk_iyy" value="0.16117211"/>
-    <xacro:property name="trunk_iyz" value="0.000048356"/>
-    <xacro:property name="trunk_izz" value="0.17460442"/>
+    <xacro:property name="trunk_mass" value="11.644"/>
+    <xacro:property name="trunk_com_x" value="0.008811"/>
+    <xacro:property name="trunk_com_y" value="0.003839"/>
+    <xacro:property name="trunk_com_z" value="0.000273"/>
+    <xacro:property name="trunk_ixx" value="0.051944892"/>
+    <xacro:property name="trunk_ixy" value="0.001703617"/>
+    <xacro:property name="trunk_ixz" value="0.000235941"/>
+    <xacro:property name="trunk_iyy" value="0.24693924"/>
+    <xacro:property name="trunk_iyz" value="0.000119783"/>
+    <xacro:property name="trunk_izz" value="0.270948307"/>
     <!-- hip (left front) -->
     <xacro:property name="hip_mass" value="1.993"/>
@@ -58,10 +79,20 @@
     <xacro:property name="hip_com_y" value="0.015144"/>
     <xacro:property name="hip_com_z" value="-0.000015"/>
-    <xacro:property name="hip_ixx" value="0.002903894"/>
-    <xacro:property name="hip_ixy" value="-0.000071850"/>
-    <xacro:property name="hip_ixz" value="-0.000001262"/>
-    <xacro:property name="hip_iyy" value="0.004907517"/>
-    <xacro:property name="hip_iyz" value="-0.00000175"/>
-    <xacro:property name="hip_izz" value="0.005586944"/>
+    <xacro:property name="hip_ixx" value="0.002446735"/>
+    <xacro:property name="hip_ixy" value="-0.00059805"/>
+    <xacro:property name="hip_ixz" value="0.000001945"/>
+    <xacro:property name="hip_iyy" value="0.003925876"/>
+    <xacro:property name="hip_iyz" value="0.000001284"/>
+    <xacro:property name="hip_izz" value="0.004148145"/>
+    <xacro:property name="hip_rotor_mass" value="0.146"/>
+    <xacro:property name="hip_rotor_com_x" value="0.0"/>
+    <xacro:property name="hip_rotor_com_y" value="0.0"/>
+    <xacro:property name="hip_rotor_com_z" value="0.0"/>
+    <xacro:property name="hip_rotor_ixx" value="0.000138702"/>
+    <xacro:property name="hip_rotor_ixy" value="0.0"/>
+    <xacro:property name="hip_rotor_ixz" value="0.0"/>
+    <xacro:property name="hip_rotor_iyy" value="0.000083352"/>
+    <xacro:property name="hip_rotor_iyz" value="0.0"/>
+    <xacro:property name="hip_rotor_izz" value="0.000083352"/>
     <!-- thigh -->
     <xacro:property name="thigh_mass" value="0.639"/>
@@ -69,10 +100,20 @@
     <xacro:property name="thigh_com_y" value="-0.003877"/>
     <xacro:property name="thigh_com_z" value="-0.048199"/>
-    <xacro:property name="thigh_ixx" value="0.005666803"/>
-    <xacro:property name="thigh_ixy" value="0.000003597"/>
-    <xacro:property name="thigh_ixz" value="0.000491446"/>
-    <xacro:property name="thigh_iyy" value="0.005847229"/>
-    <xacro:property name="thigh_iyz" value="0.000010086"/>
-    <xacro:property name="thigh_izz" value="0.000369811"/>
+    <xacro:property name="thigh_ixx" value="0.004173855"/>
+    <xacro:property name="thigh_ixy" value="0.000010284"/>
+    <xacro:property name="thigh_ixz" value="-0.000318874"/>
+    <xacro:property name="thigh_iyy" value="0.004343802"/>
+    <xacro:property name="thigh_iyz" value="0.000109233"/>
+    <xacro:property name="thigh_izz" value="0.000340136"/>
+    <xacro:property name="thigh_rotor_mass" value="0.146"/>
+    <xacro:property name="thigh_rotor_com_x" value="0.0"/>
+    <xacro:property name="thigh_rotor_com_y" value="0.0"/>
+    <xacro:property name="thigh_rotor_com_z" value="0.0"/>
+    <xacro:property name="thigh_rotor_ixx" value="0.000083352"/>
+    <xacro:property name="thigh_rotor_ixy" value="0.0"/>
+    <xacro:property name="thigh_rotor_ixz" value="0.0"/>
+    <xacro:property name="thigh_rotor_iyy" value="0.000138702"/>
+    <xacro:property name="thigh_rotor_iyz" value="0.0"/>
+    <xacro:property name="thigh_rotor_izz" value="0.000083352"/>
     <!-- calf -->
     <xacro:property name="calf_mass" value="0.207"/>
@@ -80,10 +121,20 @@
     <xacro:property name="calf_com_y" value="0.000063"/>
     <xacro:property name="calf_com_z" value="-0.142518"/>
-    <xacro:property name="calf_ixx" value="0.006341369"/>
-    <xacro:property name="calf_ixy" value="-0.000000003"/>
-    <xacro:property name="calf_ixz" value="-0.000087951"/>
-    <xacro:property name="calf_iyy" value="0.006355157"/>
-    <xacro:property name="calf_iyz" value="-0.000001336"/>
-    <xacro:property name="calf_izz" value="0.000039188"/>
+    <xacro:property name="calf_ixx" value="0.002129279"/>
+    <xacro:property name="calf_ixy" value="0.000000039"/>
+    <xacro:property name="calf_ixz" value="0.000005757"/>
+    <xacro:property name="calf_iyy" value="0.002141463"/>
+    <xacro:property name="calf_iyz" value="-0.000000516"/>
+    <xacro:property name="calf_izz" value="0.000037583"/>
+    <xacro:property name="calf_rotor_mass" value="0.132"/>
+    <xacro:property name="calf_rotor_com_x" value="0.0"/>
+    <xacro:property name="calf_rotor_com_y" value="0.0"/>
+    <xacro:property name="calf_rotor_com_z" value="0.0"/>
+    <xacro:property name="calf_rotor_ixx" value="0.000145463"/>
+    <xacro:property name="calf_rotor_ixy" value="0.0"/>
+    <xacro:property name="calf_rotor_ixz" value="0.0"/>
+    <xacro:property name="calf_rotor_iyy" value="0.000133031"/>
+    <xacro:property name="calf_rotor_iyz" value="0.0"/>
+    <xacro:property name="calf_rotor_izz" value="0.000145463"/>
     <!-- foot -->
     <xacro:property name="foot_mass" value="0.06"/>
