Commit message: first commit with new Go1 code

File: robots/aliengo_description/xacro/robot.xacro (robot description, xacro)
@@ -1,10 +1,10 @@
 <?xml version="1.0"?>
-<robot name="aliengo_description" xmlns:xacro="http://www.ros.org/wiki/xacro">
+<robot name="aliengo" xmlns:xacro="http://www.ros.org/wiki/xacro">
     <xacro:include filename="$(find aliengo_description)/xacro/const.xacro"/>
     <xacro:include filename="$(find aliengo_description)/xacro/materials.xacro"/>
     <xacro:include filename="$(find aliengo_description)/xacro/leg.xacro"/>
     <xacro:include filename="$(find aliengo_description)/xacro/gazebo.xacro"/>
-    <!-- Rollover Protection mode will add an additional stick on the top, use "true" or "false" to switch it. -->
-    <xacro:property name="rolloverProtection" value="false"/>
+    <!-- Rotor related joint and link is only for demonstrate location. -->
+    <!-- Actually, the rotor will rotate and the joint is not fixed. Reduction ratio should be considered. -->
     <!-- Debug mode will hung up the robot, use "true" or "false" to switch it. -->
     <!-- <xacro:if value="$(arg DEBUG)">
@@ -58,33 +58,4 @@
         </inertial>
     </link>
-    <xacro:if value="${(rolloverProtection == 'true')}">
-        <joint name="stick_joint" type="fixed">
-            <parent link="trunk"/>
-            <child link="stick_link"/>
-            <origin rpy="0 0 0" xyz="${0.18} 0 ${stick_length/2.0+0.08}"/>
-        </joint>
-        <link name="stick_link">
-            <visual>
-                <geometry>
-                    <cylinder length="${stick_length}" radius="${stick_radius}"/>
-                </geometry>
-                <origin rpy="0 0 0" xyz="0 0 0"/>
-                <material name="white"/>
-            </visual>
-            <collision>
-                <geometry>
-                    <cylinder length="${stick_length}" radius="${stick_radius}"/>
-                </geometry>
-                <origin rpy="0 0 0" xyz="0 0 0"/>
-            </collision>
-            <inertial>
-                <mass value="${stick_mass}"/>
-                <inertia
-                    ixx="${stick_mass / 2.0 * (stick_radius*stick_radius)}" ixy="0.0" ixz="0.0"
-                    iyy="${stick_mass / 12.0 * (3*stick_radius*stick_radius + stick_length*stick_length)}" iyz="0.0"
-                    izz="${stick_mass / 12.0 * (3*stick_radius*stick_radius + stick_length*stick_length)}"/>
-            </inertial>
-        </link>
-    </xacro:if>
     <joint name="imu_joint" type="fixed">
         <parent link="trunk"/>
@@ -96,5 +67,5 @@
             <mass value="0.001"/>
             <origin rpy="0 0 0" xyz="0 0 0"/>
-            <inertia ixx="0.0001" ixy="0" ixz="0" iyy="0.000001" iyz="0" izz="0.0001"/>
+            <inertia ixx="0.0001" ixy="0" ixz="0" iyy="0.0001" iyz="0" izz="0.0001"/>
         </inertial>
         <visual>
@@ -112,16 +83,8 @@
         </collision>
     </link>
-    <xacro:leg name="FR" mirror="-1" mirror_dae= "False" front_hind="1" front_hind_dae="True">
-        <origin rpy="0 0 0" xyz="${leg_offset_x} ${-leg_offset_y} 0"/>
-    </xacro:leg>
-    <xacro:leg name="FL" mirror="1" mirror_dae="True" front_hind="1" front_hind_dae="True">
-        <origin rpy="0 0 0" xyz="${leg_offset_x} ${leg_offset_y} 0"/>
-    </xacro:leg>
-    <xacro:leg name="RR" mirror="-1" mirror_dae="False" front_hind="-1" front_hind_dae="False">
-        <origin rpy="0 0 0" xyz="${-leg_offset_x} ${-leg_offset_y} 0"/>
-    </xacro:leg>
-    <xacro:leg name="RL" mirror="1" mirror_dae="True" front_hind="-1" front_hind_dae="False">
-        <origin rpy="0 0 0" xyz="${-leg_offset_x} ${leg_offset_y} 0"/>
-    </xacro:leg>
+    <xacro:leg name="FR" mirror="-1" mirror_dae= "False" front_hind="1"  front_hind_dae="True"  />
+    <xacro:leg name="FL" mirror="1"  mirror_dae="True"   front_hind="1"  front_hind_dae="True"  />
+    <xacro:leg name="RR" mirror="-1" mirror_dae="False"  front_hind="-1" front_hind_dae="False" />
+    <xacro:leg name="RL" mirror="1"  mirror_dae="True"   front_hind="-1" front_hind_dae="False" />
     <!-- <xacro:stairs stairs="15" xpos="0" ypos="2.0" zpos="0" /> -->
 </robot>

File: robots/laikago_description/xacro/gazebo.xacro (robot description, xacro)
@@ -1,156 +1,4 @@
 <?xml version="1.0"?>
 <robot>
-    <!-- Added by Ryan -->
-    <!--Gazebo Differential Drive Plugin-->
-  <gazebo>
-    <plugin name="diff_drive_controller" filename="libgazebo_ros_diff_drive.so">
-      <publishWheelTF>true</publishWheelTF>
-      <publishOdomTF>true</publishOdomTF>
-      <alwaysOn>true</alwaysOn>
-      <legacyMode>false</legacyMode>
-      <updateRate>40</updateRate>
-      <leftJoint>left_wheel_joint</leftJoint>
-      <rightJoint>right_wheel_joint</rightJoint>
-      <wheelSeparation>0.5</wheelSeparation>
-      <wheelDiameter>0.3</wheelDiameter>
-      <torque>20</torque>
-      <commandTopic>cmd_vel</commandTopic>
-      <odometryTopic>odom</odometryTopic>
-      <odometryFrame>odom</odometryFrame>
-      <robotBaseFrame>base</robotBaseFrame>
-    </plugin>
-  </gazebo>
-<!-- front camera -->
-  <gazebo reference="front_camera_rgb_frame">
-    <sensor type="depth" name="realsense_R200">
-      <always_on>true</always_on>
-      <visualize>false</visualize>
-      <camera>
-          <horizontal_fov>1.3439</horizontal_fov>
-          <image>
-              <width>1920</width>
-              <height>1080</height>
-              <format>R8G8B8</format>
-          </image>
-          <depth_camera></depth_camera>
-          <clip>
-              <near>0.03</near>
-              <far>100</far>
-          </clip>
-      </camera>
-      <plugin name="camera_controller" filename="libgazebo_ros_openni_kinect.so">
-        <baseline>0.2</baseline>
-        <alwaysOn>true</alwaysOn>
-        <updateRate>30.0</updateRate>
-        <cameraName>front_camera</cameraName>
-        <frameName>front_camera_link</frameName>
-        <imageTopicName>front/rgb/image_raw</imageTopicName>
-        <depthImageTopicName>front/depth/image_raw</depthImageTopicName>
-        <pointCloudTopicName>front/depth/points</pointCloudTopicName>
-        <cameraInfoTopicName>front/rgb/camera_info</cameraInfoTopicName>
-        <depthImageCameraInfoTopicName>front/depth/camera_info</depthImageCameraInfoTopicName>
-        <pointCloudCutoff>0.4</pointCloudCutoff>
-            <hackBaseline>0.07</hackBaseline>
-            <distortionK1>0.0</distortionK1>
-            <distortionK2>0.0</distortionK2>
-            <distortionK3>0.0</distortionK3>
-            <distortionT1>0.0</distortionT1>
-            <distortionT2>0.0</distortionT2>
-        <CxPrime>0.0</CxPrime>
-        <Cx>0.0</Cx>
-        <Cy>0.0</Cy>
-        <focalLength>0</focalLength>
-        <hackBaseline>0</hackBaseline>
-      </plugin>
-    </sensor>
-  </gazebo>
-<!-- rl camera -->
-  <gazebo reference="rl_camera_rgb_frame">
-    <sensor type="depth" name="realsense_R200">
-      <always_on>true</always_on>
-      <visualize>false</visualize>
-      <camera>
-          <horizontal_fov>1.3439</horizontal_fov>
-          <image>
-              <width>1920</width>
-              <height>1080</height>
-              <format>R8G8B8</format>
-          </image>
-          <depth_camera></depth_camera>
-          <clip>
-              <near>0.03</near>
-              <far>100</far>
-          </clip>
-      </camera>
-      <plugin name="camera_controller" filename="libgazebo_ros_openni_kinect.so">
-        <baseline>0.2</baseline>
-        <alwaysOn>true</alwaysOn>
-        <updateRate>30.0</updateRate>
-        <cameraName>rl_camera</cameraName>
-        <frameName>rl_camera_link</frameName>
-        <imageTopicName>rl/rgb/image_raw</imageTopicName>
-        <depthImageTopicName>rl/depth/image_raw</depthImageTopicName>
-        <pointCloudTopicName>rl/depth/points</pointCloudTopicName>
-        <cameraInfoTopicName>rl/rgb/camera_info</cameraInfoTopicName>
-        <depthImageCameraInfoTopicName>rl/depth/camera_info</depthImageCameraInfoTopicName>
-        <pointCloudCutoff>0.4</pointCloudCutoff>
-            <hackBaseline>0.07</hackBaseline>
-            <distortionK1>0.0</distortionK1>
-            <distortionK2>0.0</distortionK2>
-            <distortionK3>0.0</distortionK3>
-            <distortionT1>0.0</distortionT1>
-            <distortionT2>0.0</distortionT2>
-        <CxPrime>0.0</CxPrime>
-        <Cx>0.0</Cx>
-        <Cy>0.0</Cy>
-        <focalLength>0</focalLength>
-        <hackBaseline>0</hackBaseline>
-      </plugin>
-    </sensor>
-  </gazebo>
-  <!-- rr camera -->
-  <gazebo reference="rr_camera_rgb_frame">
-    <sensor type="depth" name="realsense_R200">
-      <always_on>true</always_on>
-      <visualize>false</visualize>
-      <camera>
-          <horizontal_fov>1.3439</horizontal_fov>
-          <image>
-              <width>1920</width>
-              <height>1080</height>
-              <format>R8G8B8</format>
-          </image>
-          <depth_camera></depth_camera>
-          <clip>
-              <near>0.03</near>
-              <far>100</far>
-          </clip>
-      </camera>
-      <plugin name="camera_controller" filename="libgazebo_ros_openni_kinect.so">
-        <baseline>0.2</baseline>
-        <alwaysOn>true</alwaysOn>
-        <updateRate>30.0</updateRate>
-        <cameraName>rr_camera</cameraName>
-        <frameName>rr_camera_link</frameName>
-        <imageTopicName>rr/rgb/image_raw</imageTopicName>
-        <depthImageTopicName>rr/depth/image_raw</depthImageTopicName>
-        <pointCloudTopicName>rr/depth/points</pointCloudTopicName>
-        <cameraInfoTopicName>rr/rgb/camera_info</cameraInfoTopicName>
-        <depthImageCameraInfoTopicName>rr/depth/camera_info</depthImageCameraInfoTopicName>
-        <pointCloudCutoff>0.4</pointCloudCutoff>
-            <hackBaseline>0.07</hackBaseline>
-            <distortionK1>0.0</distortionK1>
-            <distortionK2>0.0</distortionK2>
-            <distortionK3>0.0</distortionK3>
-            <distortionT1>0.0</distortionT1>
-            <distortionT2>0.0</distortionT2>
-        <CxPrime>0.0</CxPrime>
-        <Cx>0.0</Cx>
-        <Cy>0.0</Cy>
-        <focalLength>0</focalLength>
-        <hackBaseline>0</hackBaseline>
-      </plugin>
-    </sensor>
-  </gazebo>
     <!-- ros_control plugin -->
     <gazebo>
@@ -170,15 +18,4 @@
             </plot>
         </plugin>
-    </gazebo>
-    <gazebo>
-      <plugin name="force_based_move_controller" filename="libgazebo_ros_force_based_move.so">
-        <commandTopic>/cmd_vel_raw</commandTopic>
-        <odometryTopic>odom</odometryTopic>
-        <odometryFrame>odom</odometryFrame>
-        <odometryRate>20.0</odometryRate>
-        <robotBaseFrame>base</robotBaseFrame>
-        <yaw_velocity_p_gain>250</yaw_velocity_p_gain>
-        <publishOdometryTf>1</publishOdometryTf>
-      </plugin>
     </gazebo>
     <!-- Show the trajectory of foot. You can add another trajectory about another foot. -->

File: robots/laikago_description/xacro/robot.xacro (robot description, xacro)
@@ -1,4 +1,5 @@
 <?xml version="1.0"?>
-<robot name="laikago_description" xmlns:xacro="http://www.ros.org/wiki/xacro">
+<robot name="laikago" xmlns:xacro="http://www.ros.org/wiki/xacro">
+    <xacro:arg name="DEBUG" default="false"/>
     <xacro:include filename="$(find laikago_description)/xacro/const.xacro"/>
     <xacro:include filename="$(find laikago_description)/xacro/materials.xacro"/>
@@ -8,6 +9,5 @@
     <xacro:property name="rolloverProtection" value="false"/>
     <!-- Debug mode will hung up the robot, use "true" or "false" to switch it. -->
-    <!-- COMMENTED OUR BY RYAN -->
-<!--     <xacro:if value="$(arg DEBUG)">
+    <xacro:if value="$(arg DEBUG)">
         <link name="world"/>
         <joint name="base_static_joint" type="fixed">
@@ -16,5 +16,5 @@
             <child link="base"/>
         </joint>
-    </xacro:if>  -->
+    </xacro:if>
     <link name="base">
         <visual>
@@ -91,5 +91,5 @@
             <mass value="0.001"/>
             <origin rpy="0 0 0" xyz="0 0 0"/>
-            <inertia ixx="0.0001" ixy="0" ixz="0" iyy="0.000001" iyz="0" izz="0.0001"/>
+            <inertia ixx="0.0001" ixy="0" ixz="0" iyy="0.0001" iyz="0" izz="0.0001"/>
         </inertial>
         <visual>
@@ -107,149 +107,4 @@
         </collision>
     </link>
-<!-- Laptop Mount -->
-    <joint name="laptop_mount_joint" type="fixed">
-        <origin xyz="-0.2 0.15 0.12" rpy="0 0 0"/>
-        <parent link="trunk"/>
-        <child link="laptop_mount"/>
-    </joint>
-    <link name="laptop_mount">
-        <!-- <inertial>
-          <origin
-            xyz="-0.0017019 -8.36089999999962E-05 0.062029"
-            rpy="0 0 0" />
-          <mass
-            value="2.6502" />
-          <inertia
-            ixx="0.017805"
-            ixy="1.1578E-06"
-            ixz="4.1834E-05"
-            iyy="0.046123"
-            iyz="-4.00309999999992E-06"
-            izz="0.047358" />
-        </inertial> -->
-        <visual>
-          <origin
-            xyz="0 0 0"
-            rpy="1.5707963267949 0 0" />
-          <geometry>
-            <mesh
-              filename="package://laikago_description/meshes/laptop_mount.STL" />
-          </geometry>
-          <material
-            name="">
-            <color
-              rgba="0.79216 0.81961 0.93333 1" />
-          </material>
-        </visual>
-        <collision>
-          <origin
-            xyz="0 0 0"
-            rpy="1.5707963267949 0 0" />
-          <geometry>
-            <mesh
-              filename="package://laikago_description/meshes/laptop_mount.STL" />
-          </geometry>
-        </collision>
-    </link>
-<!-- Front Camera -->
-    <joint name="front_camera_joint" type="fixed">
-        <origin xyz="0.045 -0.05 0.25" rpy="0 0 0"/>
-        <parent link="trunk"/>
-        <child link="front_camera_link"/>
-    </joint>
-    <link name="front_camera_link">
-        <visual>
-            <origin xyz="0 0 0" rpy="1.57 0 1.57"/>
-            <geometry>
-                <mesh filename="package://laikago_description/meshes/azurekinect.dae" />
-            </geometry>
-        </visual>
-        <!-- <collision>
-            <origin xyz="0.003 0.065 0.007" rpy="0 0 0"/>
-            <geometry>
-                <box size="0.012 0.132 0.020"/>
-            </geometry>
-        </collision> -->
-    </link>
-    <joint name="front_camera_rgb_joint" type="fixed">
-        <origin xyz="0.005 0.018 0.013" rpy="0 0 0"/>
-        <parent link="front_camera_link"/>
-        <child link="front_camera_rgb_frame"/>
-    </joint>
-    <link name="front_camera_rgb_frame"/>
-    <joint name="front_camera_rgb_optical_joint" type="fixed">
-        <origin xyz="0 0 0" rpy="-1.57 0 -1.57"/>
-        <parent link="front_camera_rgb_frame"/>
-        <child link="front_camera_rgb_optical_frame"/>
-    </joint>
-    <link name="front_camera_rgb_optical_frame"/>
-<!-- RL Camera -->
-    <joint name="rl_camera_joint" type="fixed">
-        <origin xyz="0.03 0.065 0.25" rpy="0 0 -4.18879"/>
-        <parent link="trunk"/>
-        <child link="rl_camera_link"/>
-    </joint>
-    <link name="rl_camera_link">
-        <visual>
-            <origin xyz="0 0 0" rpy="1.57 0 1.57"/>
-            <geometry>
-                <mesh filename="package://laikago_description/meshes/azurekinect.dae" />
-            </geometry>
-        </visual>
-        <!-- <collision>
-            <origin xyz="0.003 0.065 0.007" rpy="0 0 0"/>
-            <geometry>
-                <box size="0.012 0.132 0.020"/>
-            </geometry>
-        </collision> -->
-    </link>
-    <joint name="rl_camera_rgb_joint" type="fixed">
-        <origin xyz="0.005 0.018 0.013" rpy="0 0 0"/>
-        <parent link="rl_camera_link"/>
-        <child link="rl_camera_rgb_frame"/>
-    </joint>
-    <link name="rl_camera_rgb_frame"/>
-    <joint name="rl_camera_rgb_optical_joint" type="fixed">
-        <origin xyz="0 0 0" rpy="-1.57 0 -1.57"/>
-        <parent link="rl_camera_rgb_frame"/>
-        <child link="rl_camera_rgb_optical_frame"/>
-    </joint>
-    <link name="rl_camera_rgb_optical_frame"/>
-<!-- RR Camera -->
-    <joint name="rr_camera_joint" type="fixed">
-        <origin xyz="-0.065 -0.015 0.25" rpy="0 0 4.18879"/>
-        <parent link="trunk"/>
-        <child link="rr_camera_link"/>
-    </joint>
-    <link name="rr_camera_link">
-        <visual>
-            <origin xyz="0 0 0" rpy="1.57 0 1.57"/>
-            <geometry>
-                <mesh filename="package://laikago_description/meshes/azurekinect.dae" />
-            </geometry>
-        </visual>
-        <!-- <collision>
-            <origin xyz="0.003 0.065 0.007" rpy="0 0 0"/>
-            <geometry>
-                <box size="0.012 0.132 0.020"/>
-            </geometry>
-        </collision> -->
-    </link>
-    <joint name="rr_camera_rgb_joint" type="fixed">
-        <origin xyz="0.005 0.018 0.013" rpy="0 0 0"/>
-        <parent link="rr_camera_link"/>
-        <child link="rr_camera_rgb_frame"/>
-    </joint>
-    <link name="rr_camera_rgb_frame"/>
-    <joint name="rr_camera_rgb_optical_joint" type="fixed">
-        <origin xyz="0 0 0" rpy="-1.57 0 -1.57"/>
-        <parent link="rr_camera_rgb_frame"/>
-        <child link="rr_camera_rgb_optical_frame"/>
-    </joint>
-    <link name="rr_camera_rgb_optical_frame"/>
-    <xacro:include filename="$(find velodyne_description)/urdf/VLP-16.urdf.xacro"/>
-    <VLP-16 parent="base" name="velodyne" topic="lidar_points" hz="10" samples="1024" gpu="false" lasers="16" max_range="100">
-        <origin xyz="0.0075 0.0 0.3025" rpy="0 0 0" />
-    </VLP-16>
     <xacro:leg name="FR" mirror="-1" mirror_dae="False" front_hind="1" front_hind_dae="True">
         <origin rpy="0 0 0" xyz="${leg_offset_x} ${-leg_offset_y} 0"/>
